Commit message: feat: second commit

File: catkin_ws/src/puzzlebot_sim/urdf/puzzlebot.urdf.xacro (robot description, xacro)
@@ -2,5 +2,4 @@
 <robot xmlns:xacro="http://www.ros.org/wiki/xacro" name="puzzlebot">
     <xacro:property name="cdeg" value="1.57" /> <!-- Turn 90 deg -->
-    <link name="base_footprint" />
     <xacro:property name="constant" value="0.083" /> <!-- 1/12 -->
     <xacro:property name="mass" value="0.710" />
@@ -8,6 +7,13 @@
     <xacro:property name="height" value="0.29" />
     <xacro:property name="depth" value="0.17" />
+    <link name="base_link" />
+    <joint name="base_joint" type="fixed">
+        <!-- <origin xyz="0.0 0.0 0.05" rpy="0.0 0.0 0.0"/> -->
+        <parent link="base_link"/>
+        <child link="chassis"/>
+        <!-- <axis xyz="0.0 0.0 1.0"/> -->
+    </joint>
     <!-- ROBOT CHASSIS-->
-    <link name="base_link">
+    <link name="chassis">
         <inertial>
             <origin xyz="0.0 0.0 0.0" rpy="${cdeg} 0.0 ${cdeg}"/>
@@ -34,10 +40,4 @@
         </collision>
     </link>
-    <joint name="base_joint" type="fixed">
-        <origin xyz="0.0 0.0 0.05" rpy="0.0 0.0 0.0"/>
-        <parent link="base_footprint"/>
-        <child link="base_link"/>
-        <axis xyz="0.0 0.0 1.0"/>
-    </joint>
     <!-- ROBOT WHEELS -->
     <xacro:macro name="wheel" params="name x y deg">
@@ -67,5 +67,5 @@
         <joint name="wheel_${name}_joint" type="continuous">
             <origin xyz="${x} ${y} 0.0" rpy="0.0 0.0 0.0"/>
-            <parent link="base_link"/>
+            <parent link="chassis"/>
             <child link="wheel_${name}_link"/>
             <axis xyz="0.0 0.0 1.0"/>
