Commit message: feat: Add MiniC_2 final

File: catkin_ws_8/src/puzzlebot_sim/urdf/puzzlebot_sim.urdf (robot description, URDF)
Before this commit: robot PuzzleBot, 4 links, 3 joints
Links:
- removed link base_link
- removed link chassis
- removed link left_wheel
- removed link right_wheel
- added link base_link_rviz
- added link chassis_rviz; visual mesh filename=file://$(find puzzlebot_sim)/meshes/MCR2_1000_13_Chassis.stl
- added link left_wheel_rviz; visual mesh filename=file://$(find puzzlebot_sim)/meshes/MCR2_1000_1_1_Wheel_Cou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
- added link right_wheel_rviz; visual mesh filename=file://$(find puzzlebot_sim)/meshes/MCR2_1000_1_1_Wheel_Cou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
Joints:
- joint base_link_to_chassis: child chassis -> chassis_rviz; parent base_link -> base_link_rviz
- joint base_to_left_w: child left_wheel -> left_wheel_rviz; parent base_link -> base_link_rviz
- joint base_to_right_w: child right_wheel -> right_wheel_rviz; parent base_link -> base_link_rviz
