Commit message: feat: mini challenge 1

File: catkin_ws/src/puzzlebot_gazebo/urdf/macros.xacro (robot description, xacro)
@@ -1,25 +1,25 @@
 <?xml version="1.0"?>
 <robot xmlns:xacro="http://www.ros.org/wiki/xacro">
-<!-- note to self: modify this to add wheel as left and right with -->
-    <xacro:macro name="box_inertia" params="m x y z">
-            <inertia
-          ixx="${m/12.0 * (y*y + z*z)}" ixy="0.0" ixz="0.0"
-          iyy="${m/12.0 * (z*z + x*x)}" iyz="0.0"
-          izz="${m/12.0 * (y*y + x*x)}"/>
-        <!--  <inertia
-          ixx="0.001" ixy="0.0" ixz="0.0"
-          iyy="0.001" iyz="0.0"
-          izz="0.001"/>-->
-    </xacro:macro>
-    <xacro:macro name="wheel_inertia" params="r l m">
-              <!--<inertia  ixx="${m*(3*r*r+l*l)/12}" ixy = "0" ixz = "0"
-                iyy="${m*(3*r*r+l*l)/12}" iyz = "0"
-                izz="${m*(r*r)/2}" />-->
-              <!--  <inertia  ixx="0.00001" ixy = "0" ixz = "0"
-                iyy="0.00001" iyz = "0"
-                izz="0.00001" />-->
-               <inertia  ixx="${(m/12)*(3*((r*r)+((r/4)*(r/4)))+(l*l))}" ixy="0" ixz="0"
-                iyy="${(m/12)*(3*((r*r)+((r/4)*(r/4)))+(l*l))}" iyz="0"
-                izz="${(m/2)*(r*r+(r/4)*(r/4))}" />
-    </xacro:macro>
+  <!-- note to self: modify this to add wheel as left and right with -->
+  <xacro:macro name="box_inertia" params="m x y z">
+    <inertia
+      ixx="${m/12.0 * (y*y + z*z)}" ixy="0.0" ixz="0.0"
+      iyy="${m/12.0 * (z*z + x*x)}" iyz="0.0"
+      izz="${m/12.0 * (y*y + x*x)}"/>
+      <!--  <inertia
+      ixx="0.001" ixy="0.0" ixz="0.0"
+      iyy="0.001" iyz="0.0"
+      izz="0.001"/>-->
+  </xacro:macro>
+  <xacro:macro name="wheel_inertia" params="r l m">
+    <!--<inertia  ixx="${m*(3*r*r+l*l)/12}" ixy = "0" ixz = "0"
+      iyy="${m*(3*r*r+l*l)/12}" iyz = "0"
+      izz="${m*(r*r)/2}" />-->
+    <!--  <inertia  ixx="0.00001" ixy = "0" ixz = "0"
+      iyy="0.00001" iyz = "0"
+      izz="0.00001" />-->
+      <inertia  ixx="${(m/12)*(3*((r*r)+((r/4)*(r/4)))+(l*l))}" ixy="0" ixz="0"
+      iyy="${(m/12)*(3*((r*r)+((r/4)*(r/4)))+(l*l))}" iyz="0"
+      izz="${(m/2)*(r*r+(r/4)*(r/4))}" />
+  </xacro:macro>
 </robot>

File: catkin_ws/src/puzzlebot_gazebo/urdf/puzzlebot.xacro (robot description, xacro)
@@ -8,132 +8,132 @@
 <xacro:include filename="$(find puzzlebot_gazebo)/urdf/macros.xacro" />
 <!-- Dummy link to fiz robot chassis -->
-  <link name="base_link">
-    <pose>0 0 0 0 0 0</pose>
-  </link>
-  <joint name="base_link_to_chassis" type="fixed">
+	<link name="base_link">
+    	<pose>0 0 0 0 0 0</pose>
+  	</link>
+  	<joint name="base_link_to_chassis" type="fixed">
 	   <parent link="base_link"/>
 	   <child link="chassis"/>
-  </joint>
-  <link name="chassis">
-    <pose>0 0 0 0 0 0</pose>
-    <visual>
-    <!-- box only
-      <origin xyz="0 0 0" rpy="0 0 0"/>
-          <geometry>
-          	  <box size="${chassisX} ${chassisY} ${chassisZ}"/>
-          </geometry> -->
-      <!-- with mesh  -->
-      <origin xyz="0 0 0" rpy="${PI/2} 0 ${PI/2}"/>
-          <geometry>
-          	 <mesh filename="file://${mesh_chassis}"/>
-          </geometry>
-    </visual>
-    <collision name="collision_chassis">
-    	<origin rpy="0 0 0" xyz="0 0 0"/>
-          <geometry>
-            	 <box size="${chassisX} ${chassisY} ${chassisZ}"/>
-          </geometry>
-    </collision>
-    <inertial>
-      <mass value="${chassisMass}"/>
-      <xacro:box_inertia m="${chassisMass}" x="${chassisX}" y="${chassisY}" z="${chassisZ}" />
-    </inertial>
-   <!-- agregar caster wheel en frame -->
-    <collision>
-	    <origin xyz="-0.095 0 -0.0425" rpy="0 0 0"/>
-		  <geometry>
-		     <sphere radius="${casterRadius}"/>
-		  </geometry>
-		        <surface>
-	      <friction>
-	         <ode>
-	          <slip1>0.0</slip1>
-	          <slip2>0.0</slip2>
-	         </ode>
-	      </friction>
-      </surface>
-	  </collision>
-	  <visual>
-      <origin xyz="-0.095 0 -0.0425" rpy="0 0 0"/>
-          <geometry>
-          	   <sphere radius="${casterRadius}"/>
-          </geometry>
-    </visual>
-  </link>
+  	</joint>
+  	<link name="chassis">
+    	<pose>0 0 0 0 0 0</pose>
+    	<visual>
+			<!-- box only
+			<origin xyz="0 0 0" rpy="0 0 0"/>
+			<geometry>
+				<box size="${chassisX} ${chassisY} ${chassisZ}"/>
+			</geometry> -->
+			<!-- with mesh  -->
+			<origin xyz="0 0 0" rpy="${PI/2} 0 ${PI/2}"/>
+			<geometry>
+				<mesh filename="file://${mesh_chassis}"/>
+			</geometry>
+    	</visual>
+		<collision name="collision_chassis">
+			<origin rpy="0 0 0" xyz="0 0 0"/>
+			<geometry>
+				<box size="${chassisX} ${chassisY} ${chassisZ}"/>
+			</geometry>
+		</collision>
+		<inertial>
+			<mass value="${chassisMass}"/>
+			<xacro:box_inertia m="${chassisMass}" x="${chassisX}" y="${chassisY}" z="${chassisZ}" />
+		</inertial>
+		<!-- Agregar caster wheel en frame -->
+		<collision>
+			<origin xyz="-0.095 0 -0.0425" rpy="0 0 0"/>
+			<geometry>
+				<sphere radius="${casterRadius}"/>
+			</geometry>
+			<surface>
+				<friction>
+					<ode>
+						<slip1>0.0</slip1>
+						<slip2>0.0</slip2>
+					</ode>
+				</friction>
+			</surface>
+		</collision>
+		<visual>
+			<origin xyz="-0.095 0 -0.0425" rpy="0 0 0"/>
+				<geometry>
+				<sphere radius="${casterRadius}"/>
+				</geometry>
+		</visual>
+  	</link>
     <!--RIGHT WHEEL -->
 	<link name="right_wheel">
-	  <visual>
-	  	<origin xyz="0 0 0" rpy="-${PI/2} 0 0" />
-	    <geometry>
-	      <!-- with mesh-->
-	      	<mesh filename="file://${mesh_wheel}"/>
-	    	<!-- cylinder only
-	    	<cylinder length="${wheelHeight}" radius="${wheelRadius}"/> -->
-	    </geometry>
-	  </visual>
-	  <collision>
-		  <origin xyz="0 0 0 " rpy="-${PI/2} 0 0"/>
-			  <geometry>
-			     <cylinder length="${wheelHeight}" radius="${wheelRadius}" />
-			  </geometry>
-	  </collision>
-	  <inertial>
-		  <mass value="${wheelMass}"/>
-		  <origin xyz="0 0 0" rpy="${PI/2} 0 0"/>
-		  <xacro:wheel_inertia r="${wheelRadius}" l="${wheelHeight}" m="${wheelMass}"/>
-	  </inertial>
+		<visual>
+	  		<origin xyz="0 0 0" rpy="-${PI/2} 0 0" />
+	    	<geometry>
+				<!-- with mesh-->
+				<mesh filename="file://${mesh_wheel}"/>
+				<!-- cylinder only
+				<cylinder length="${wheelHeight}" radius="${wheelRadius}"/> -->
+	    	</geometry>
+	  	</visual>
+	  	<collision>
+		  	<origin xyz="0 0 0 " rpy="-${PI/2} 0 0"/>
+			<geometry>
+			    <cylinder length="${wheelHeight}" radius="${wheelRadius}" />
+			</geometry>
+	  	</collision>
+	 	<inertial>
+			<mass value="${wheelMass}"/>
+			<origin xyz="0 0 0" rpy="${PI/2} 0 0"/>
+			<xacro:wheel_inertia r="${wheelRadius}" l="${wheelHeight}" m="${wheelMass}"/>
+	  	</inertial>
 	</link>
     <!-- LEFT WHEEL -->
 	<link name="left_wheel">
-	  <visual>
-	    <geometry>
-        <!-- with mesh-->
-	      	<mesh filename="file://${mesh_wheel}"/>
-	    	<!-- cylinder only
-	    	<cylinder length="${wheelHeight}" radius="${wheelRadius}"/> -->
-	    </geometry>
-	    <origin xyz="0 0 0" rpy="${PI/2} 0 0" />
-	  </visual>
-	  <collision>
+		<visual>
+			<geometry>
+			<!-- with mesh-->
+				<mesh filename="file://${mesh_wheel}"/>
+				<!-- cylinder only
+				<cylinder length="${wheelHeight}" radius="${wheelRadius}"/> -->
+			</geometry>
+			<origin xyz="0 0 0" rpy="${PI/2} 0 0" />
+		</visual>
+	  	<collision>
 		  <origin xyz="0 0 0" rpy="${PI/2} 0 0" />
 		  <geometry>
 		     <cylinder length="${wheelHeight}" radius="${wheelRadius}"/>
 		  </geometry>
-	  </collision>
-	  <inertial>
+	  	</collision>
+	  	<inertial>
 		  <mass value="${wheelMass}"/>
 		  <origin xyz="0 0 0" rpy="${PI/2} 0 0"/>
 		  <xacro:wheel_inertia r="${wheelRadius}" l="${wheelHeight}" m="${wheelMass}" />
-	  </inertial>
+	  	</inertial>
 	</link>
-	 <!-- CAMERA-->
-	 <link name="camera">
-		    <inertial>
-		    	    <origin rpy="0 0 0" xyz="0 0 0"/>
-		          <mass value="0.007"/>
-		          <inertia ixx="0.166667" ixy="0" ixz="0" iyy="0.166667" iyz="0" izz="0.166667"/>
-		          <!-- ad camera inertia -->
-		    </inertial>
-		    <collision name="collision_chassis">
-		    	    <origin rpy="0 0 0" xyz="0 0 0"/>
-		          <geometry>
-		               <box size="0.05 0.01 0.06" />
-		          </geometry>
-		    </collision>
-		    <visual>
-		    	    <!-- box only
-		    	    <origin rpy="$0 0 ${PI/2}" xyz="0 0 0"/>
-		          <geometry>
-		          	<box size="0.05 0.01 0.06" />
-		          </geometry>-->
-		         <!-- with mesh-->
-		          <origin rpy="${PI/2} 0 ${PI/2}" xyz="0 0 0"/>
-		          <geometry>
-		          	<mesh filename="file://${mesh_camera}"/>
-		          </geometry>
-		    </visual>
-  </link>
-<!-- JOINTS  -->
-  <joint name="base_to_right_w" type="continuous">
+	<!-- CAMERA-->
+	<link name="camera">
+		<inertial>
+			<origin rpy="0 0 0" xyz="0 0 0"/>
+			<mass value="0.007"/>
+			<inertia ixx="0.166667" ixy="0" ixz="0" iyy="0.166667" iyz="0" izz="0.166667"/>
+			<!-- ad camera inertia -->
+		</inertial>
+		<collision name="collision_chassis">
+			<origin rpy="0 0 0" xyz="0 0 0"/>
+			<geometry>
+				<box size="0.05 0.01 0.06" />
+			</geometry>
+		</collision>
+		<visual>
+			<!-- box only
+			<origin rpy="$0 0 ${PI/2}" xyz="0 0 0"/>
+			<geometry>
+			<box size="0.05 0.01 0.06" />
+			</geometry>-->
+			<!-- with mesh-->
+			<origin rpy="${PI/2} 0 ${PI/2}" xyz="0 0 0"/>
+			<geometry>
+			<mesh filename="file://${mesh_camera}"/>
+			</geometry>
+		</visual>
+  	</link>
+	<!-- JOINTS  -->
+  	<joint name="base_to_right_w" type="continuous">
 	  <parent link="chassis" />
 	  <child link="right_wheel" />
@@ -151,30 +151,30 @@
 		<joint_properties damping="0.0" friction="0.0"/>-->
 	</joint>
-<!---->
-<joint name="camera_to_base" type="fixed">
+	<!---->
+	<joint name="camera_to_base" type="fixed">
 	  <parent link="chassis" />
 	  <child link="camera" />
 	  <origin xyz="0.09 0 0.048" rpy= "0.0 0.24 0.0" />
-  </joint>
-<!-- TRANSMISSIONS (For a more complex model and it represents actuator attributes) -->
-<transmission name="right_wheel_trans">
-    <type>transmission_interface/SimpleTransmission</type>
-    <joint name="base_to_right_w">
-    	<hardwareInterface>hardware_interface/EffortJointInterface</hardwareInterface>
-    </joint>
-    <actuator name="right_wheel_motor">
-      <mechanicalReduction>34</mechanicalReduction>
-       <hardwareInterface>hardware_interface/EffortJointInterface</hardwareInterface>
-    </actuator>
-  </transmission>
-<transmission name="left_wheel_trans">
-    <type>transmission_interface/SimpleTransmission</type>
-    <joint name="base_to_left_w">
-    	<hardwareInterface>hardware_interface/EffortJointInterface</hardwareInterface>
-    </joint>
-    <actuator name="left_wheel_motor">
-      <mechanicalReduction>34</mechanicalReduction>
-      <hardwareInterface>hardware_interface/EffortJointInterface</hardwareInterface>
-    </actuator>
-</transmission>
+  	</joint>
+	<!-- TRANSMISSIONS (For a more complex model and it represents actuator attributes) -->
+	<transmission name="right_wheel_trans">
+		<type>transmission_interface/SimpleTransmission</type>
+		<joint name="base_to_right_w">
+			<hardwareInterface>hardware_interface/EffortJointInterface</hardwareInterface>
+		</joint>
+		<actuator name="right_wheel_motor">
+		<mechanicalReduction>34</mechanicalReduction>
+		<hardwareInterface>hardware_interface/EffortJointInterface</hardwareInterface>
+		</actuator>
+	</transmission>
+	<transmission name="left_wheel_trans">
+		<type>transmission_interface/SimpleTransmission</type>
+		<joint name="base_to_left_w">
+			<hardwareInterface>hardware_interface/EffortJointInterface</hardwareInterface>
+		</joint>
+		<actuator name="left_wheel_motor">
+		<mechanicalReduction>34</mechanicalReduction>
+		<hardwareInterface>hardware_interface/EffortJointInterface</hardwareInterface>
+		</actuator>
+	</transmission>
 </robot>

File: catkin_ws/src/puzzlebot_rviz/urdf/puzzlebot.urdf.xacro (robot description, xacro)
@@ -26,5 +26,5 @@
             <origin xyz="0.0 0.0 0.0" rpy="${cdeg} 0.0 ${cdeg}"/>
             <geometry>
-                <mesh filename="package://puzzlebot_sim/meshes/chassis.stl" scale="1 1 1"/>
+                <mesh filename="package://puzzlebot_rviz/meshes/chassis.stl" scale="1 1 1"/>
             </geometry>
             <material name="red">
@@ -36,5 +36,5 @@
             <origin xyz="0.0 0.0 0.0" rpy="${cdeg} 0.0 ${cdeg}"/>
             <geometry>
-                <mesh filename="package://puzzlebot_sim/meshes/chassis.stl" scale="1 1 1"/>
+                <mesh filename="package://puzzlebot_rviz/meshes/chassis.stl" scale="1 1 1"/>
             </geometry>
         </collision>
@@ -51,5 +51,5 @@
                 <origin xyz="0.0 0.0 0.0" rpy="0.0 ${cdeg} ${deg}"/>
                 <geometry>
-                     <mesh filename="package://puzzlebot_sim/meshes/wheel_coupler.stl" scale="1 1 1"/>
+                     <mesh filename="package://puzzlebot_rviz/meshes/wheel_coupler.stl" scale="1 1 1"/>
                 </geometry>
                 <material name="blue">
@@ -61,5 +61,5 @@
                 <origin xyz="0.0 0.0 0.0" rpy="0.0 ${cdeg} ${deg}"/>
                 <geometry>
-                    <mesh filename="package://puzzlebot_sim/meshes/wheel_coupler.stl" scale="1 1 1"/>
+                    <mesh filename="package://puzzlebot_rviz/meshes/wheel_coupler.stl" scale="1 1 1"/>
                 </geometry>
             </collision>
