Commit message: feat: Delete puzzlebot_sim_8 and puzzlebot_rviz_8

File: catkin_ws/src/puzzlebot_gazebo/urdf/macros.xacro (robot description, xacro)
@@ -1,25 +1,25 @@
 <?xml version="1.0"?>
 <robot xmlns:xacro="http://www.ros.org/wiki/xacro">
-  <!-- note to self: modify this to add wheel as left and right with -->
-  <xacro:macro name="box_inertia" params="m x y z">
-    <inertia
-      ixx="${m/12.0 * (y*y + z*z)}" ixy="0.0" ixz="0.0"
-      iyy="${m/12.0 * (z*z + x*x)}" iyz="0.0"
-      izz="${m/12.0 * (y*y + x*x)}"/>
-      <!--  <inertia
-      ixx="0.001" ixy="0.0" ixz="0.0"
-      iyy="0.001" iyz="0.0"
-      izz="0.001"/>-->
-  </xacro:macro>
-  <xacro:macro name="wheel_inertia" params="r l m">
-    <!--<inertia  ixx="${m*(3*r*r+l*l)/12}" ixy = "0" ixz = "0"
-      iyy="${m*(3*r*r+l*l)/12}" iyz = "0"
-      izz="${m*(r*r)/2}" />-->
-    <!--  <inertia  ixx="0.00001" ixy = "0" ixz = "0"
-      iyy="0.00001" iyz = "0"
-      izz="0.00001" />-->
-      <inertia  ixx="${(m/12)*(3*((r*r)+((r/4)*(r/4)))+(l*l))}" ixy="0" ixz="0"
-      iyy="${(m/12)*(3*((r*r)+((r/4)*(r/4)))+(l*l))}" iyz="0"
-      izz="${(m/2)*(r*r+(r/4)*(r/4))}" />
-  </xacro:macro>
+<!-- note to self: modify this to add wheel as left and right with -->
+    <xacro:macro name="box_inertia" params="m x y z">
+            <inertia
+          ixx="${m/12.0 * (y*y + z*z)}" ixy="0.0" ixz="0.0"
+          iyy="${m/12.0 * (z*z + x*x)}" iyz="0.0"
+          izz="${m/12.0 * (y*y + x*x)}"/>
+        <!--  <inertia
+          ixx="0.001" ixy="0.0" ixz="0.0"
+          iyy="0.001" iyz="0.0"
+          izz="0.001"/>-->
+    </xacro:macro>
+    <xacro:macro name="wheel_inertia" params="r l m">
+              <!--<inertia  ixx="${m*(3*r*r+l*l)/12}" ixy = "0" ixz = "0"
+                iyy="${m*(3*r*r+l*l)/12}" iyz = "0"
+                izz="${m*(r*r)/2}" />-->
+              <!--  <inertia  ixx="0.00001" ixy = "0" ixz = "0"
+                iyy="0.00001" iyz = "0"
+                izz="0.00001" />-->
+               <inertia  ixx="${(m/12)*(3*((r*r)+((r/4)*(r/4)))+(l*l))}" ixy="0" ixz="0"
+                iyy="${(m/12)*(3*((r*r)+((r/4)*(r/4)))+(l*l))}" iyz="0"
+                izz="${(m/2)*(r*r+(r/4)*(r/4))}" />
+    </xacro:macro>
 </robot>

File: catkin_ws/src/puzzlebot_gazebo/urdf/puzzlebot.xacro (robot description, xacro)
@@ -1,47 +1,47 @@
-<?xml version="1.0" ?>
+<?xml version="1.0"?>
 <!-- PuzzleBot differential drive -->
 <robot name="puzzlebot" xmlns:xacro="http://www.ros.org/wiki/xacro">
-<!-- files for gazebo costumization -->
-<xacro:include filename="$(find puzzlebot_gazebo)/urdf/materials.xacro" />
-<xacro:include filename="$(find puzzlebot_gazebo)/urdf/parameters.xacro" />
-<xacro:include filename="$(find puzzlebot_gazebo)/urdf/puzzlebot.gazebo" />
-<xacro:include filename="$(find puzzlebot_gazebo)/urdf/macros.xacro" />
-<!-- Dummy link to fiz robot chassis -->
+	<!-- files for gazebo costumization -->
+	<xacro:include filename="$(find puzzlebot_gazebo)/urdf/materials.xacro" />
+	<xacro:include filename="$(find puzzlebot_gazebo)/urdf/parameters.xacro" />
+	<xacro:include filename="$(find puzzlebot_gazebo)/urdf/puzzlebot.gazebo" />
+	<xacro:include filename="$(find puzzlebot_gazebo)/urdf/macros.xacro" />
+	<!-- Dummy link to fiz robot chassis -->
 	<link name="base_link">
-    	<pose>0 0 0 0 0 0</pose>
-  	</link>
-  	<joint name="base_link_to_chassis" type="fixed">
-	   <parent link="base_link"/>
-	   <child link="chassis"/>
-  	</joint>
-  	<link name="chassis">
-    	<pose>0 0 0 0 0 0</pose>
-    	<visual>
+		<pose>0 0 0 0 0 0</pose>
+	</link>
+	<joint name="base_link_to_chassis" type="fixed">
+		<parent link="base_link" />
+		<child link="chassis" />
+	</joint>
+	<link name="chassis">
+		<pose>0 0 0 0 0 0</pose>
+		<visual>
 			<!-- box only
-			<origin xyz="0 0 0" rpy="0 0 0"/>
-			<geometry>
-				<box size="${chassisX} ${chassisY} ${chassisZ}"/>
-			</geometry> -->
+      <origin xyz="0 0 0" rpy="0 0 0"/>
+          <geometry>
+          	  <box size="${chassisX} ${chassisY} ${chassisZ}"/>
+          </geometry> -->
 			<!-- with mesh  -->
-			<origin xyz="0 0 0" rpy="${PI/2} 0 ${PI/2}"/>
-			<geometry>
-				<mesh filename="file://${mesh_chassis}"/>
-			</geometry>
-    	</visual>
+			<origin xyz="0 0 0" rpy="${PI/2} 0 ${PI/2}" />
+			<geometry>
+				<mesh filename="file://${mesh_chassis}" />
+			</geometry>
+		</visual>
 		<collision name="collision_chassis">
-			<origin rpy="0 0 0" xyz="0 0 0"/>
-			<geometry>
-				<box size="${chassisX} ${chassisY} ${chassisZ}"/>
-			</geometry>
-		</collision>
-		<inertial>
-			<mass value="${chassisMass}"/>
+			<origin rpy="0 0 0" xyz="0 0 0" />
+			<geometry>
+				<box size="${chassisX} ${chassisY} ${chassisZ}" />
+			</geometry>
+		</collision>
+		<inertial>
+			<mass value="${chassisMass}" />
 			<xacro:box_inertia m="${chassisMass}" x="${chassisX}" y="${chassisY}" z="${chassisZ}" />
 		</inertial>
-		<!-- Agregar caster wheel en frame -->
-		<collision>
-			<origin xyz="-0.095 0 -0.0425" rpy="0 0 0"/>
-			<geometry>
-				<sphere radius="${casterRadius}"/>
+		<!-- agregar caster wheel en frame -->
+		<collision>
+			<origin xyz="-0.095 0 ${-0.0435}" rpy="0 0 0" />
+			<geometry>
+				<sphere radius="${casterRadius}" />
 			</geometry>
 			<surface>
@@ -55,106 +55,169 @@
 		</collision>
 		<visual>
-			<origin xyz="-0.095 0 -0.0425" rpy="0 0 0"/>
-				<geometry>
-				<sphere radius="${casterRadius}"/>
-				</geometry>
-		</visual>
-  	</link>
-    <!--RIGHT WHEEL -->
+			<origin xyz="-0.095 0 -0.0435" rpy="0 0 0" />
+			<geometry>
+				<sphere radius="${casterRadius}" />
+			</geometry>
+		</visual>
+	</link>
+	<!--RIGHT
+	WHEEL -->
 	<link name="right_wheel">
 		<visual>
-	  		<origin xyz="0 0 0" rpy="-${PI/2} 0 0" />
-	    	<geometry>
+			<origin xyz="0 0 0" rpy="-${PI/2} 0 0" />
+			<geometry>
 				<!-- with mesh-->
-				<mesh filename="file://${mesh_wheel}"/>
+				<mesh filename="file://${mesh_wheel}" />
 				<!-- cylinder only
-				<cylinder length="${wheelHeight}" radius="${wheelRadius}"/> -->
-	    	</geometry>
-	  	</visual>
-	  	<collision>
-		  	<origin xyz="0 0 0 " rpy="-${PI/2} 0 0"/>
-			<geometry>
-			    <cylinder length="${wheelHeight}" radius="${wheelRadius}" />
-			</geometry>
-	  	</collision>
-	 	<inertial>
-			<mass value="${wheelMass}"/>
-			<origin xyz="0 0 0" rpy="${PI/2} 0 0"/>
-			<xacro:wheel_inertia r="${wheelRadius}" l="${wheelHeight}" m="${wheelMass}"/>
-	  	</inertial>
-	</link>
-    <!-- LEFT WHEEL -->
+	    	<cylinder length="${wheelHeight}" radius="${wheelRadius}"/> -->
+			</geometry>
+		</visual>
+		<collision>
+			<origin xyz="0 0 0 " rpy="-${PI/2} 0 0" />
+			<geometry>
+				<cylinder length="${wheelHeight}" radius="${wheelRadius+0.0010032}" />
+			</geometry>
+		</collision>
+		<inertial>
+			<mass value="${wheelMass}" />
+			<origin xyz="0 0 0" rpy="${PI/2} 0 0" />
+			<xacro:wheel_inertia r="${wheelRadius}" l="${wheelHeight}" m="${wheelMass}" />
+		</inertial>
+	</link>
+	<!-- LEFT WHEEL -->
 	<link name="left_wheel">
 		<visual>
 			<geometry>
-			<!-- with mesh-->
-				<mesh filename="file://${mesh_wheel}"/>
+				<!-- with mesh-->
+				<mesh filename="file://${mesh_wheel}" />
 				<!-- cylinder only
-				<cylinder length="${wheelHeight}" radius="${wheelRadius}"/> -->
-			</geometry>
-			<origin xyz="0 0 0" rpy="${PI/2} 0 0" />
-		</visual>
-	  	<collision>
-		  <origin xyz="0 0 0" rpy="${PI/2} 0 0" />
-		  <geometry>
-		     <cylinder length="${wheelHeight}" radius="${wheelRadius}"/>
-		  </geometry>
-	  	</collision>
-	  	<inertial>
-		  <mass value="${wheelMass}"/>
-		  <origin xyz="0 0 0" rpy="${PI/2} 0 0"/>
-		  <xacro:wheel_inertia r="${wheelRadius}" l="${wheelHeight}" m="${wheelMass}" />
-	  	</inertial>
+	    	<cylinder length="${wheelHeight}" radius="${wheelRadius}"/> -->
+			</geometry>
+			<origin xyz="0 0 0" rpy="${PI/2} 0 0" />
+		</visual>
+		<collision>
+			<origin xyz="0 0 0" rpy="${PI/2} 0 0" />
+			<geometry>
+				<cylinder length="${wheelHeight}" radius="${wheelRadius+0.0010032}" />
+			</geometry>
+		</collision>
+		<inertial>
+			<mass value="${wheelMass}" />
+			<origin xyz="0 0 0" rpy="${PI/2} 0 0" />
+			<xacro:wheel_inertia r="${wheelRadius}" l="${wheelHeight}" m="${wheelMass}" />
+		</inertial>
 	</link>
 	<!-- CAMERA-->
 	<link name="camera">
 		<inertial>
-			<origin rpy="0 0 0" xyz="0 0 0"/>
-			<mass value="0.007"/>
-			<inertia ixx="0.166667" ixy="0" ixz="0" iyy="0.166667" iyz="0" izz="0.166667"/>
+			<origin rpy="0 0 0" xyz="0 0 0" />
+			<mass value="0.007" />
+			<inertia ixx="0.166667" ixy="0" ixz="0" iyy="0.166667" iyz="0" izz="0.166667" />
 			<!-- ad camera inertia -->
 		</inertial>
 		<collision name="collision_chassis">
-			<origin rpy="0 0 0" xyz="0 0 0"/>
-			<geometry>
-				<box size="0.05 0.01 0.06" />
+			<origin rpy="0 0 0" xyz="0 0 0" />
+			<geometry>
+				<box size="0.07 0.01 0.06" />
 			</geometry>
 		</collision>
 		<visual>
 			<!-- box only
-			<origin rpy="$0 0 ${PI/2}" xyz="0 0 0"/>
-			<geometry>
-			<box size="0.05 0.01 0.06" />
-			</geometry>-->
+		    	    <origin rpy="$0 0 ${PI/2}" xyz="0 0 0"/>
+		          <geometry>
+		          	<box size="0.05 0.01 0.06" />
+		          </geometry>-->
 			<!-- with mesh-->
-			<origin rpy="${PI/2} 0 ${PI/2}" xyz="0 0 0"/>
-			<geometry>
-			<mesh filename="file://${mesh_camera}"/>
-			</geometry>
-		</visual>
-  	</link>
+			<origin rpy="${PI/2} 0 ${PI/2}" xyz="0 0 0" />
+			<geometry>
+				<mesh filename="file://${mesh_camera}" />
+			</geometry>
+		</visual>
+	</link>
+	<link name="camera_frame_optical" />
+	<!-- LIDAR-->
+	<link name="lidar">
+		<inertial>
+			<mass value="0.1" />
+			<origin xyz="0 0 0" />
+			<inertia ixx="0.01" ixy="0.0" ixz="0.0"
+					 iyy="0.01" iyz="0.0"
+					 izz="0.01" />
+		</inertial>
+		<!-- <visual>
+			<origin xyz=" 0 0 0 " rpy="0 0 0" />
+			<geometry>
+				<cylinder length="0.05" radius="0.05"/>
+			</geometry>
+			<material name="black"/>
+		</visual> -->
+		<collision>
+			<origin xyz="-0.06 0.0 -0.04" rpy="0 0 0" />
+			<geometry>
+				<cylinder length="0.01" radius="0.05"/>
+			</geometry>
+		</collision>
+        <visual>
+			<origin rpy="${PI/2} 0 0" xyz="0.07 -0.013 -0.04" />
+            <geometry>
+                <mesh filename="file://${mesh_lidar}" />
+            </geometry>
+        </visual>
+		<![CDATA[
+        <collision>
+			<origin rpy="0 0 0" xyz="0 0 0" />
+			<!-- <geometry>
+				<box size="1000 1000 0.01" />
+			</geometry> -->
+			<geometry>
+				<!-- <mesh filename="file://${mesh_lidar}" /> -->
+				<!-- <box size="0.01 0.01 0.01" /> -->
+				<cylinder length="0.01" radius="0.5" />
+			</geometry>
+        </collision>
+        <!-- <inertial_cylinder mass="0.1" length="0.04" radius="0.05">
+            <origin xyz="0 0 0" rpy="0 0 0"/>
+        </inertial_cylinder> -->
+		<inertial>
+			<origin rpy="0 0 0" xyz="0 0 0" />
+			<mass value="0.000" />
+			<inertia ixx="0.166667" ixy="0" ixz="0" iyy="0.166667" iyz="0" izz="0.166667" />
+			<!-- ad camera inertia -->
+		</inertial>]]>
+    </link>
 	<!-- JOINTS  -->
-  	<joint name="base_to_right_w" type="continuous">
-	  <parent link="chassis" />
-	  <child link="right_wheel" />
-	  <origin xyz="0.05 -0.09 0.0" />
+	<joint name="base_to_right_w" type="continuous">
+		<parent link="chassis" />
+		<child link="right_wheel" />
+		<origin xyz="0.05 -0.09 0.0" />
 		<axis xyz="0 1 0" rpy="0 0 0" />
-	<!--	<limit effort="100" velocity="100"/>
+		<!--	<limit effort="100" velocity="100"/>
 		<joint_properties damping="0.0" friction="0.0"/>-->
 	</joint>
 	<joint name="base_to_left_w" type="continuous">
-	  <parent link="chassis" />
-	  <child link="left_wheel" />
-	  <origin xyz="0.05 0.09 0" />
-	  <axis xyz="0 1 0" rpy="0 0 0" />
-		<!--<limit effort="100" velocity="100"/>
+		<parent link="chassis" />
+		<child link="left_wheel" />
+		<origin xyz="0.05 0.09 0" />
+		<axis xyz="0 1 0" rpy="0 0 0" />
+		<!--<limit
+		effort="100" velocity="100"/>
 		<joint_properties damping="0.0" friction="0.0"/>-->
 	</joint>
 	<!---->
 	<joint name="camera_to_base" type="fixed">
-	  <parent link="chassis" />
-	  <child link="camera" />
-	  <origin xyz="0.09 0 0.048" rpy= "0.0 0.24 0.0" />
-  	</joint>
+		<parent link="chassis" />
+		<child link="camera" />
+		<origin xyz="0.1 0 0.048" rpy="0.0 0 0.0" />
+	</joint>
+	<joint name="camera_frame_to_camera" type="fixed">
+		<origin xyz="0 0 0" rpy="${-pi/2} 0 ${-pi/2}" />
+		<parent link="camera" />
+		<child link="camera_frame_optical" />
+	</joint>
+	<joint name="lidar_to_base" type="fixed">
+        <parent link="chassis"/>
+        <child link="lidar"/>
+        <origin xyz="0.05 0 0.115" rpy="0 0 ${PI}"/>
+    </joint>
 	<!-- TRANSMISSIONS (For a more complex model and it represents actuator attributes) -->
 	<transmission name="right_wheel_trans">
@@ -164,6 +227,6 @@
 		</joint>
 		<actuator name="right_wheel_motor">
-		<mechanicalReduction>34</mechanicalReduction>
-		<hardwareInterface>hardware_interface/EffortJointInterface</hardwareInterface>
+			<mechanicalReduction>34</mechanicalReduction>
+			<hardwareInterface>hardware_interface/EffortJointInterface</hardwareInterface>
 		</actuator>
 	</transmission>
@@ -174,6 +237,6 @@
 		</joint>
 		<actuator name="left_wheel_motor">
-		<mechanicalReduction>34</mechanicalReduction>
-		<hardwareInterface>hardware_interface/EffortJointInterface</hardwareInterface>
+			<mechanicalReduction>34</mechanicalReduction>
+			<hardwareInterface>hardware_interface/EffortJointInterface</hardwareInterface>
 		</actuator>
 	</transmission>
